File: KiCAD/Display Adapters/Display Adapters.kicad_sch (KiCad schematic)
At the start: 3 parts, among them J1 20455-040E-76, J2 G46M2023201BTWEU, J3 XT30PW-M

Commit message: source pcb done
Parts:
- removed J1: 20455-040E-76, 20455-040E-76:IPEX_20455-040E-76, symbol 20455-040E-76:20455-040E-76
- removed J2: G46M2023201BTWEU, G46M2023201BTWEU:AMPHENOL_G46M2023201BTWEU, symbol G46M2023201BTWEU:G46M2023201BTWEU
- removed J3: XT30PW-M, XT30PW-M:AMASS_XT30PW-M, symbol XT30PW-M:XT30PW-M
Connections:
- no-connect marks 4 -> 0
Other:
- added sheet sink (sink.kicad_sch)
- added sheet source (source.kicad_sch)
