File: KiCAD/Display Adapters/Display Adapters.kicad_pcb (KiCad board)
At the start: 4 copper layers, 38 x 29.6 mm, 8 parts, among them J1 20455-040E-76, J2 G46M2013201AWEU, J3 XT30PW_2_2_-M.G.B, J4 XT30PW_2_2_-M.G.B, J5 G46M2013201AWEU, J6 20455-040E-76

Commit message: work on sink side
Parts:
- removed H1, H2: MountingHole_Pad, MountingHole:MountingHole_2.2mm_M2_DIN965_Pad_TopBottom
- removed J1: 20455-040E-76, SnapEDA:IPEX_20455-040E-76
- removed J2: G46M2013201AWEU, SnapEDA:AMPHENOL_G46M2013201AWEU
- removed J3: XT30PW_2_2_-M.G.B, SnapEDA:AMASS_XT30PW_2_2_-M.G.B
- added C2: 1uF, Capacitor_SMD:C_0603_1608Metric_Pad1.08x0.95mm_HandSolder, F.Cu at (153.7, 41.8)
- added C3: 1uF, Capacitor_SMD:C_0603_1608Metric_Pad1.08x0.95mm_HandSolder, F.Cu at (147.2, 41.8)
- moved J4 22.9 mm to (156.8, 65.5)
- moved J5 7.84 mm to (141.8, 63.6)
- moved J6 7.75 mm to (146.9, 46.1)
Routing:
- net +5V: track 64.6 -> 41.9 mm
- net EDP_HPD: track 44.9 -> 23.5 mm
- net GND: track 24.1 -> 16.3 mm, vias 21 -> 11
- net AUX_N: track 55.8 -> 48.8 mm
- net AUX_P: track 55.5 -> 48.5 mm
- net 0_EDP_TX_N: track 26.8 -> 20.5 mm
- net 0_EDP_TX_P: track 26.8 -> 20.5 mm
- net BLK_OFF_N: track 23.5 -> 29.5 mm
- net 2_EDP_TX_N: track 26.7 -> 21.5 mm
- net 2_EDP_TX_P: track 26.6 -> 21.5 mm
- net 3_EDP_TX_P: track 25.7 -> 20.6 mm
- net 3_EDP_TX_N: track 25.7 -> 20.6 mm
- net +3.3V: track 13.1 -> 10.2 mm
- net BLK_PWM_LCD: track 25.8 -> 24.0 mm
- net 1_EDP_TX_P: track 19.9 -> 20.8 mm
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Other:
- board size 38 x 29.6 mm -> 35.1 x 30.5 mm
- board text removed: "Source: EDP -> DP"
