File: KiCAD/Display Adapters/sink.kicad_sch (KiCad schematic)
At the start: 5 parts, among them J4 XT30PW_2_2_-M.G.B, J5 G46M2013201AWEU, J6 20455-040E-76

Commit message: work on sink side
Parts:
- C2, C3: footprint (none) -> Capacitor_SMD:C_0603_1608Metric_Pad1.08x0.95mm_HandSolder
Changed lines of the file:
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@@
+				)
+			)
+			(project "sink"
+				(path "/fce918aa-4ffb-4ad3-b88d-35171bd3e360"
+					(reference "#PWR0110")
+					(unit 1)
 				)
 			)
@@
 				)
 			)
+			(project "sink"
+				(path "/fce918aa-4ffb-4ad3-b88d-35171bd3e360"
+					(reference "J3")
+					(unit 1)
+				)
+			)
 		)
 	)
@@
 				)
 			)
+			(project "sink"
+				(path "/fce918aa-4ffb-4ad3-b88d-35171bd3e360"
+					(reference "#PWR0103")
+					(unit 1)
+				)
+			)
 		)
 	)
@@
 			)
 		)
-		(property "Footprint" ""
+		(property "Footprint" "Capacitor_SMD:C_0603_1608Metric_Pad1.08x0.95mm_HandSolder"
 			(at 199.39 113.03 0)
 			(effects
@@
 			(project "Display Adapters"
 				(path "/d30881c9-2e5b-4846-8f12-42ee4af8a2cb/fcc0638b-2731-4e5e-82a0-257b53736c6a"
+					(reference "C2")
+					(unit 1)
+				)
+			)
+			(project "sink"
+				(path "/fce918aa-4ffb-4ad3-b88d-35171bd3e360"
 					(reference "C2")
 					(unit 1)
@@
 				)
 			)
+			(project "sink"
+				(path "/fce918aa-4ffb-4ad3-b88d-35171bd3e360"
+					(reference "#PWR0109")
+					(unit 1)
+				)
+			)
 		)
 	)
@@
 			)
 		)
-		(property "Footprint" ""
+		(property "Footprint" "Capacitor_SMD:C_0603_1608Metric_Pad1.08x0.95mm_HandSolder"
 			(at 185.42 95.25 0)
 			(effects
@@
 				(path "/d30881c9-2e5b-4846-8f12-42ee4af8a2cb/fcc0638b-2731-4e5e-82a0-257b53736c6a"
 					(reference "C3")
+					(unit 1)
+				)
+			)
+			(project "sink"
+				(path "/fce918aa-4ffb-4ad3-b88d-35171bd3e360"
+					(reference "C1")
 					(unit 1)
 				)
@@
 				(path "/d30881c9-2e5b-4846-8f12-42ee4af8a2cb/fcc0638b-2731-4e5e-82a0-257b53736c6a"
 					(reference "J4")
+					(unit 1)
+				)
+			)
+			(project "sink"
+				(path "/fce918aa-4ffb-4ad3-b88d-35171bd3e360"
+					(reference "J1")
 					(unit 1)
 				)
@@
 				)
 			)
+			(project "sink"
+				(path "/fce918aa-4ffb-4ad3-b88d-35171bd3e360"
+					(reference "#PWR0107")
+					(unit 1)
+				)
+			)
 		)
 	)
@@
 				(path "/d30881c9-2e5b-4846-8f12-42ee4af8a2cb/fcc0638b-2731-4e5e-82a0-257b53736c6a"
 					(reference "#PWR017")
+					(unit 1)
+				)
+			)
+			(project "sink"
+				(path "/fce918aa-4ffb-4ad3-b88d-35171bd3e360"
+					(reference "#PWR0104")
 					(unit 1)
 				)
@@
 				)
 			)
+			(project "sink"
+				(path "/fce918aa-4ffb-4ad3-b88d-35171bd3e360"
+					(reference "#PWR0105")
+					(unit 1)
+				)
+			)
 		)
 	)
@@
 				)
 			)
+			(project "sink"
+				(path "/fce918aa-4ffb-4ad3-b88d-35171bd3e360"
+					(reference "#PWR0106")
+					(unit 1)
+				)
+			)
 		)
 	)
@@
 				)
 			)
+			(project "sink"
+				(path "/fce918aa-4ffb-4ad3-b88d-35171bd3e360"
+					(reference "#PWR0108")
+					(unit 1)
+				)
+			)
 		)
 	)
@@
 				)
 			)
+			(project "sink"
+				(path "/fce918aa-4ffb-4ad3-b88d-35171bd3e360"
+					(reference "#PWR0102")
+					(unit 1)
+				)
+			)
 		)
 	)
@@
 				(path "/d30881c9-2e5b-4846-8f12-42ee4af8a2cb/fcc0638b-2731-4e5e-82a0-257b53736c6a"
 					(reference "J5")
+					(unit 1)
+				)
+			)
+			(project "sink"
+				(path "/fce918aa-4ffb-4ad3-b88d-35171bd3e360"
+					(reference "J2")
 					(unit 1)
 				)
@@
 				)
 			)
+			(project "sink"
+				(path "/fce918aa-4ffb-4ad3-b88d-35171bd3e360"
+					(reference "#PWR0101")
+					(unit 1)
+				)
+			)
 		)
 	)
+	(sheet_instances
+		(path "/"
+			(page "1")
+		)
+	)
+	(embedded_fonts no)
 )
