File: KiCAD/Display Adapters/source/source.kicad_sch (KiCad schematic)
At the start: 5 parts, among them J1 20455-040E-76, J2 XT30PW_2_2_-M.G.B, J3 G46M2013201AWEU

Commit message: use full sized dp instead
Parts:
- removed J3: G46M2013201AWEU, SnapEDA:AMPHENOL_G46M2013201AWEU, symbol G46M2013201AWEU:G46M2013201AWEU
- added J2: 47272-0001, SnapEDA:MOLEX_47272-0001, symbol 47272-0001:47272-0001
- renumbered J2 to J3
Connections:
- net +3.3V: now also J2.20
- net 0_EDP_TX_N: now also J2.3
- net 0_EDP_TX_P: now also J2.1
- net 1_EDP_TX_N: now also J2.6
- net 1_EDP_TX_P: now also J2.4
- net 2_EDP_TX_N: now also J2.9
- net 2_EDP_TX_P: now also J2.7
- net 3_EDP_TX_N: now also J2.12
- net 3_EDP_TX_P: now also J2.10
- net AUX_N: now also J2.17
- net AUX_P: now also J2.15
- net BLK_OFF_N: now also J3.S1; no longer J3.S2
- net BLK_PWM_LCD: now also J3.S2; no longer J3.S1
- net EDP_HPD: now also J2.18
- net GND: now also J2.11, J2.13, J2.14, J2.16, J2.19, J2.2, J2.5, J2.8, J2.S1 (SHIELD), J2.S2 (SHIELD), J2.S3 (SHIELD), J2.S4 (SHIELD)
Other:
- note added: "Displayport Connector"
- note removed: "Mini Displayport Connector"
