File: KiCAD/Keyboard/frameortho.kicad_pcb (KiCad board)
At the start: 2 copper layers, 276 x 105 mm, 138 parts, among them SW1 SW_Push, SW2 SW_Push, U1 RP2040, U2 W25Q128JVS, U3 XC6206PxxxMR, Y1 12 MHz 18pF

Commit message: aaaaaaaaaaaaaaaaaa
Other:
- board text added: "JLCJLCJLCJLC"

Commit message: make board smaller
Parts:
- removed the H8 at (322.8, 99.4)
- added H10: MountingHole_Pad, MountingHole:MountingHole_2.2mm_M2_DIN965_Pad_TopBottom, F.Cu at (315.2, 90.0)
- added H11: MountingHole_Pad, MountingHole:MountingHole_2.2mm_M2_DIN965_Pad_TopBottom, F.Cu at (191.6, 140.6)
- added H12: MountingHole_Pad, MountingHole:MountingHole_2.2mm_M2_DIN965_Pad_TopBottom, F.Cu at (232.9, 140.6)
- added H13: MountingHole_Pad, MountingHole:MountingHole_2.2mm_M2_DIN965_Pad_TopBottom, F.Cu at (109.2, 90.0)
- added H9: MountingHole_Pad, MountingHole:MountingHole_2.2mm_M2_DIN965_Pad_TopBottom, F.Cu at (315.2, 175.0)
- moved H6 76.0 mm to (109.2, 175.0)
- moved H3 0.62 mm to (232.9, 152.6)
- moved H1 0.62 mm to (191.6, 152.6)
- moved C7 0.31 mm to (212.2, 103.3)
- moved C12 0.09 mm to (211.6, 105.4)
- renumbered H7 to H5, H9 to H7, H10 to H8, 3.3V to TP23, 1.1V to TP24, GND to TP25
Routing:
- net GND: track 108.9 -> 101.7 mm, vias 38 -> 39
- net +3V3: track 120.8 -> 121.6 mm
Other:
- board size 276 x 105 mm -> 226 x 105 mm
